File: ICN6211_breakout.kicad_pcb (KiCad board)
At the start: 2 copper layers, 42 x 34.8 mm, 23 parts, among them J1 Conn_STM32MP1, J2 Conn_VDD1, J3 Conn_VDD2, J4 Conn_PWR, J5 Conn_GPIO, U1 ICN6211

Commit message: Rev 2
Parts:
- removed J1: Conn_STM32MP1, Connector_FFC-FPC:Molex_200528-0200_1x20-1MP_P1.00mm_Horizontal
- removed J4: Conn_PWR, Connector_PinHeader_2.54mm:PinHeader_1x03_P2.54mm_Vertical
- added J10: Conn_DSI, Connector_FFC-FPC:TE_2-1734839-6_1x26-1MP_P0.5mm_Horizontal, F.Cu at (155.8, 60.0)
- added TP10: TP_SCL, TestPoint:TestPoint_Pad_D1.0mm, B.Cu at (155.6, 61.6)
- J5: footprint Connector_PinHeader_2.54mm:PinHeader_2x16_P2.54mm_Vertical -> Connector_PinHeader_2.54mm:PinHeader_2x20_P2.54mm_Vertical
- TP1: value TP_STM_INT -> TP_5V
- TP2: value TP_STM_TE -> TP_DATA18
- TP3: value TP_STM_BL -> TP_DATA19
- TP4: value TP_STM_RST -> TP_DATA20
- TP5: value TP_STM_VDD -> TP_DATA21
- TP6: value TP_DSI_D2+ -> TP_DATA22
- TP7: value TP_DSI_D2- -> TP_DATA23
- TP8: value TP_DSI_D3+ -> TP_REF_CLK
- TP9: value TP_DSI_D3- -> TP_SDA; moved to B.Cu
- moved TP2 40.9 mm to (127.0, 62.2), turned to 45 degrees
- moved TP3 38.0 mm to (129.5, 62.2), turned to 45 degrees
- moved TP5 35.3 mm to (134.6, 62.2), turned to 45 degrees
- moved TP4 34.9 mm to (132.2, 62.2), turned to 45 degrees
- moved TP6 34.1 mm to (137.2, 62.2), turned to 135 degrees
- moved TP7 33.1 mm to (139.7, 62.2), turned to 135 degrees
- moved TP9 26.7 mm to (153.0, 61.6)
- moved TP8 26.1 mm to (143.5, 53.3)
- moved R1 19.6 mm to (136.8, 51.6), turned to -135 degrees
- moved R2 18.7 mm to (137.8, 52.6), turned to 45 degrees
- moved TP1 11.0 mm to (165.6, 37.4), turned to 0 degrees
- moved J2 10.0 mm to (117.5, 53.0)
- moved J3 10.0 mm to (117.5, 49.0)
- moved C3 6.78 mm to (135.0, 50.0)
- moved C4 6.78 mm to (134.0, 49.0)
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Connections:
- J5 pad 1: /DATA0 -> +3V3
- J5 pad 10: /DATA21 -> /DATA9
- J5 pad 11: /DATA5 -> /DATA11
- J5 pad 12: /DE -> /SPI_CS
- J5 pad 13: /DATA6 -> /TOUCH_INT
- J5 pad 14: /PCLK -> GND
- J5 pad 15: /DATA7 -> /DATA2
- J5 pad 16: /HSYNC -> /DATA3
- J5 pad 17: /DATA8 -> +3V3
- J5 pad 18: /VSYNC -> /DATA4
- J5 pad 19: /DATA9 -> /SDA
- J5 pad 2: /REF_CLK -> +5V
- J5 pad 20: /DATA20 -> GND
- J5 pad 21: /DATA10 -> /DATA17
- J5 pad 22: /DATA19 -> /DATA5
- J5 pad 23: /DATA11 -> /SCL
- J5 pad 24: /DATA18 -> /DATA16
- J5 pad 25: /DATA12 -> GND
- J5 pad 26: /DATA17 -> /DATA15
- J5 pad 27: /DATA13 -> /PCLK
- J5 pad 28: /DATA16 -> /DE
- J5 pad 29: /DATA14 -> /DATA13
- J5 pad 3: /DATA1 -> /VSYNC
- J5 pad 30: /DATA15 -> GND
- J5 pad 31: GND -> /DATA14
- J5 pad 32: +3V3 -> /DATA6
- J5 pad 4: /EN -> +5V
- J5 pad 5: /DATA2 -> /HSYNC
- J5 pad 6: /DATA23 -> GND
- J5 pad 7: /DATA3 -> /DATA12
- J5 pad 8: /DATA22 -> /DATA8
- J5 pad 9: /DATA4 -> GND
- R1 pad 2: VDD2 -> VDD1
- R2 pad 1: VDD2 -> VDD1
- TP1 pad 1: Net-(J1-Pad17) -> +5V
- TP2 pad 1: Net-(J1-Pad18) -> /DATA18
- TP3 pad 1: Net-(J1-Pad19) -> /DATA19
- TP4 pad 1: Net-(J1-Pad20) -> /DATA20
- TP5 pad 1: Net-(J1-Pad14) -> /DATA21
- TP6 pad 1: Net-(TP6-Pad1) -> /DATA22
- TP7 pad 1: Net-(TP7-Pad1) -> /DATA23
- TP8 pad 1: Net-(TP8-Pad1) -> /REF_CLK
- TP9 pad 1: Net-(TP9-Pad1) -> /SDA
- U1 pad 20: Net-(TP6-Pad1) -> /DSI_D2+
- U1 pad 21: Net-(TP7-Pad1) -> /DSI_D2-
- U1 pad 22: Net-(TP8-Pad1) -> /DSI_D3+
- U1 pad 23: Net-(TP9-Pad1) -> /DSI_D3-
Routing:
- net +3V3: track 23.0 -> 86.4 mm, vias 0 -> 1
- net /SPI_MOSI: track 0.00 -> 53.2 mm
- net /BL_CTRL: track 0.00 -> 52.0 mm, vias 0 -> 2
- net /TOUCH_INT: track 0.00 -> 29.2 mm, vias 0 -> 2
- net +1V8: track 12.6 -> 41.3 mm, vias 0 -> 1
- net /DATA1: track 21.1 -> 48.7 mm, vias 0 -> 1
- net /SDA: track 33.2 -> 60.2 mm, vias 2 -> 3
- net /DSI_D3-: track 0.00 -> 25.4 mm
- net /SPI_CS: track 0.00 -> 25.3 mm, vias 0 -> 2
- net /REF_CLK: track 29.2 -> 4.12 mm, vias 2 -> 0
- net /DSI_D3+: track 0.00 -> 25.1 mm
- net /DSI_D2-: track 0.00 -> 24.2 mm
- net /DSI_D2+: track 0.00 -> 23.9 mm
- net Net-(TP9-Pad1): track 20.7 -> 0.00 mm, vias 2 -> 0
- net Net-(TP8-Pad1): track 20.1 -> 0.00 mm, vias 2 -> 0
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- added copper zone on GND, net GND
- removed copper zone on B.Cu, net GND
- removed copper zone on F.Cu, net GND
Other:
- board size 42 x 34.8 mm -> 52 x 34.8 mm
- copper layers 2 -> 4
- board text added: "5V"
- board text added: "BKLT"
- board text added: "DSI to RGB LCD by arturo182 Mar 2020"
- board text added: "MOSI"
- board text added: "SCL"
- board text added: "SDA"
- board text added: "T_INT"
- board text added: "VDD1"
- board text added: "VDD2"
- board text added: "~CS~"
- board text removed: "BL"
- board text removed: "D2+"
- board text removed: "D2-"
- board text removed: "D3+"
- board text removed: "D3-"
- board text removed: "DSI to RGB LCD by arturo182 Feb 2020"
- board text removed: "EN"
- board text removed: "FROM STM"
- board text removed: "INT"
- board text removed: "RST"
- board text removed: "TE"
- board text removed: "VDD"
- board text removed: "VDSI"
- board text removed: "VRGB VI2C"
