File: ICN6211_breakout.sch (KiCad schematic (older format))
At the start: 23 parts, among them J1 Conn_STM32MP1, J2 Conn_VDD1, J3 Conn_VDD2, J4 Conn_PWR, J5 Conn_GPIO, U1 ICN6211

Commit message: Rev 2
Parts:
- removed J1: Conn_STM32MP1, Connector_FFC-FPC:Molex_200528-0200_1x20-1MP_P1.00mm_Horizontal, symbol Connector_Generic:Conn_01x20
- removed J4: Conn_PWR, Connector_PinHeader_2.54mm:PinHeader_1x03_P2.54mm_Vertical, symbol Connector_Generic:Conn_01x03
- added J10: Conn_DSI, Connector_FFC-FPC:TE_2-1734839-6_1x26-1MP_P0.5mm_Horizontal, symbol Connector_Generic:Conn_01x26
- added TP10: TP_SCL, TestPoint:TestPoint_Pad_D1.0mm, symbol Connector:TestPoint
- J5: footprint Connector_PinHeader_2.54mm:PinHeader_2x16_P2.54mm_Vertical -> Connector_PinHeader_2.54mm:PinHeader_2x20_P2.54mm_Vertical; symbol Connector_Generic:Conn_02x16_Odd_Even -> Connector_Generic:Conn_02x20_Odd_Even
- TP1: value TP_STM_INT -> TP_5V
- TP2: value TP_STM_TE -> TP_DATA18
- TP3: value TP_STM_BL -> TP_DATA19
- TP4: value TP_STM_RST -> TP_DATA20
- TP5: value TP_STM_VDD -> TP_DATA21
- TP6: value TP_DSI_D2+ -> TP_DATA22
- TP7: value TP_DSI_D2- -> TP_DATA23
- TP8: value TP_DSI_D3+ -> TP_REF_CLK
- TP9: value TP_DSI_D3- -> TP_SDA
Connections:
- net +1V8: now also J10.2 (Pin_2)
- net +3V3: now also J5.1 (Pin_1), J5.17 (Pin_17), J10.1 (Pin_1); no longer J5.32 (Pin_32)
- net DATA0: now also J5.38 (Pin_38); no longer J5.1 (Pin_1)
- net DATA1: now also J5.40 (Pin_40); no longer J5.3 (Pin_3)
- net DATA10: now also J5.36 (Pin_36); no longer J5.21 (Pin_21)
- net DATA11: now also J5.11 (Pin_11); no longer J5.23 (Pin_23)
- net DATA12: now also J5.7 (Pin_7); no longer J5.25 (Pin_25)
- net DATA13: now also J5.29 (Pin_29); no longer J5.27 (Pin_27)
- net DATA14: now also J5.31 (Pin_31); no longer J5.29 (Pin_29)
- net DATA15: now also J5.26 (Pin_26); no longer J5.30 (Pin_30)
- net DATA16: now also J5.24 (Pin_24); no longer J5.28 (Pin_28)
- net DATA17: now also J5.21 (Pin_21); no longer J5.26 (Pin_26)
- net DATA18: now also TP2.1; no longer J5.24 (Pin_24)
- net DATA19: now also TP3.1; no longer J5.22 (Pin_22)
- net DATA2: now also J5.15 (Pin_15); no longer J5.5 (Pin_5)
- net DATA20: now also TP4.1; no longer J5.20 (Pin_20)
- net DATA21: now also TP5.1; no longer J5.10 (Pin_10)
- net DATA22: now also TP6.1; no longer J5.8 (Pin_8)
- net DATA23: now also TP7.1; no longer J5.6 (Pin_6)
- net DATA3: now also J5.16 (Pin_16); no longer J5.7 (Pin_7)
- net DATA4: now also J5.18 (Pin_18); no longer J5.9 (Pin_9)
- net DATA5: now also J5.22 (Pin_22); no longer J5.11 (Pin_11)
- net DATA6: now also J5.32 (Pin_32); no longer J5.13 (Pin_13)
- net DATA7: now also J5.33 (Pin_33); no longer J5.15 (Pin_15)
- net DATA8: now also J5.8 (Pin_8); no longer J5.17 (Pin_17)
- net DATA9: now also J5.10 (Pin_10); no longer J5.19 (Pin_19)
- net DE: now also J5.28 (Pin_28); no longer J5.12 (Pin_12)
- net DSI_CLK+: now also J10.13 (Pin_13)
- net DSI_CLK-: now also J10.14 (Pin_14)
- net DSI_D0+: now also J10.16 (Pin_16)
- net DSI_D0-: now also J10.17 (Pin_17)
- net DSI_D1+: now also J10.19 (Pin_19)
- net DSI_D1-: now also J10.20 (Pin_20)
- net EN: now also J10.4 (Pin_4); no longer J5.4 (Pin_4)
- net GND: now also J5.14 (Pin_14), J5.20 (Pin_20), J5.25 (Pin_25), J5.30 (Pin_30), J5.34 (Pin_34), J5.39 (Pin_39), J5.6 (Pin_6), J5.9 (Pin_9), J10.12 (Pin_12), J10.15 (Pin_15), J10.18 (Pin_18), J10.21 (Pin_21), J10.24 (Pin_24), J10.3 (Pin_3), J10.9 (Pin_9); no longer J5.31 (Pin_31)
- net HSYNC: now also J5.5 (Pin_5); no longer J5.16 (Pin_16)
- net PCLK: now also J5.27 (Pin_27); no longer J5.14 (Pin_14)
- net REF_CLK: now also TP8.1; no longer J5.2 (Pin_2)
- net SCL: now also J5.23 (Pin_23), J10.11 (Pin_11), TP10.1
- net SDA: now also J5.19 (Pin_19), TP9.1, J10.10 (Pin_10)
- net VDD1: now also R1.2, R2.1
- net VDD2: no longer R1.2, R2.1
- net VSYNC: now also J5.3 (Pin_3); no longer J5.18 (Pin_18)
- net DSI_D2+: now reaches U1.20 (DSI_D2+)
- net DSI_D2+: now also J10.22 (Pin_22); no longer TP6.1
- net DSI_D2-: now reaches U1.21 (DSI_D2-)
- net DSI_D2-: now also J10.23 (Pin_23); no longer TP7.1
- net DSI_D3+: now reaches U1.22 (DSI_D3+)
- net DSI_D3+: now also J10.25 (Pin_25); no longer TP8.1
- net DSI_D3-: now reaches U1.23 (DSI_D3-)
- net DSI_D3-: now also J10.26 (Pin_26); no longer TP9.1
- net +5V: now reaches TP1.1
- net +5V: now also J5.2 (Pin_2), J5.4 (Pin_4)
- new net BL_CTRL: J10.5 (Pin_5), J5.35 (Pin_35)
- new net SPI_CS: J10.7 (Pin_7), J5.12 (Pin_12)
- new net SPI_MOSI: J10.6 (Pin_6), J5.37 (Pin_37)
- new net TOUCH_INT: J10.8 (Pin_8), J5.13 (Pin_13)
Other:
- note added: "0.5mm pitch"
- note added: "1.8V"
- note added: "VDD1"
- moved on the sheet: C1, C2, C3, C4, C5, C6, R1, R2, U1
